Commit message: 新增躯干rviz 模型

File: ros2_ws/src/marvin_mesh_sim/urdf/marvin_mesh_hands.urdf (robot description, URDF)
Before this commit: robot marvin_mesh_dual_arm_hands, 44 links, 43 joints
Links:
- added link Gento_Luna_Leg_J1_Link, mass 6.042; collision box size=0.1560000032 0.3305 0.173999995; visual mesh filename=package://marvin_mesh_sim/meshes/other/Gento_Luna_Leg_J1_Li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
- added link Gento_Luna_Leg_J2_Link, mass 6.04185968; collision box size=0.1560000032 0.455994368 0.1924978942; visual mesh filename=package://marvin_mesh_sim/meshes/other/Gento_Luna_Leg_J2_Li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
- added link Gento_Luna_Leg_J3_Link, mass 4.67121672; collision box size=0.1560000032 0.455999992 0.203901082; visual mesh filename=package://marvin_mesh_sim/meshes/other/Gento_Luna_Leg_J3_Li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
- added link Gento_Luna_Leg_J4_Link, mass 5.90046349; collision box size=0.1530000046 0.1419976502 0.1070000008; visual mesh filename=package://marvin_mesh_sim/meshes/other/Gento_Luna_Leg_J4_Li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
- added link Gento_Luna_Leg_J5_Link, mass 3.76177572; collision box size=0.174997896 0.245499998 0.292241388; visual mesh filename=package://marvin_mesh_sim/meshes/other/Gento_Luna_Leg_J5_Li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
- added link Gento_Luna_Leg_J6_Link, mass 7.69392497; collision box size=0.2670964 0.250500142 0.366451964; visual mesh filename=package://marvin_mesh_sim/meshes/other/Gento_Luna_Leg_J6_Li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
- added link Head_J1_Link, mass 0.7216; collision box size=0.0869999974 0.1185000018 0.0970000028; visual mesh filename=package://marvin_mesh_sim/meshes/other/Head_J1_Link.STL
- added link Head_J2_Link, mass 2.3905; collision box size=0.1669688746 0.1482419 0.212378994; visual mesh filename=package://marvin_mesh_sim/meshes/other/Head_J2_Link.STL
- link base_link: mass None -> 90.8; geometry collision box size=0.669569076 0.547638148 0.380585744; visual mesh filename=package://marvin_mesh_sim/meshes/base/Underpan_Base_link.STL
Joints:
- removed joint world_to_fixture
- added joint Gento_Luna_Leg_J1_Joint: type revolute, parent base_link, child Gento_Luna_Leg_J1_Link, origin xyz=0 0 0.1 rpy=1.57080000079 -6.749156789e-12 1.57080000079, axis 0 0 1, limit lower=-0.191986218 upper=0.191986218 effort=2.0 velocity=2.0
- added joint Gento_Luna_Leg_J2_Joint: type revolute, parent Gento_Luna_Leg_J1_Link, child Gento_Luna_Leg_J2_Link, origin xyz=0 0.165 0 rpy=3.14159265359 -1.57079265408 3.14159265359, axis 0 0 1, limit lower=-1.57079633 upper=1.57079633 effort=2.0 velocity=2.0
- added joint Gento_Luna_Leg_J3_Joint: type revolute, parent Gento_Luna_Leg_J2_Link, child Gento_Luna_Leg_J3_Link, origin xyz=0 0.3 0 rpy=0 -0 0, axis 0 0 1, limit lower=-2.44346095 upper=1.04719755 effort=2.0 velocity=2.0
- added joint Gento_Luna_Leg_J4_Joint: type revolute, parent Gento_Luna_Leg_J3_Link, child Gento_Luna_Leg_J4_Link, origin xyz=0 0.3 0 rpy=0 -0 0, axis 0 0 1, limit lower=-0.959931089 upper=1.91986218 effort=2.0 velocity=2.0
- added joint Gento_Luna_Leg_J5_Joint: type revolute, parent Gento_Luna_Leg_J4_Link, child Gento_Luna_Leg_J5_Link, origin xyz=0 0 0 rpy=3.14159265359 1.57079265408 3.14159265359, axis 0 0 1, limit lower=-0.523598776 upper=0.523598776 effort=2.0 velocity=2.0
- added joint Gento_Luna_Leg_J6_Joint: type revolute, parent Gento_Luna_Leg_J5_Link, child Gento_Luna_Leg_J6_Link, origin xyz=0 0 0 rpy=1.57079448988 -1.57079265279 3.14159081658, axis 0 0 1, limit lower=-2.96705973 upper=2.96705973 effort=2.0 velocity=2.0
- added joint Head_J1_joint: type revolute, parent Gento_Luna_Leg_J6_Link, child Head_J1_Link, origin xyz=-0.013496 0 0.49898 rpy=1.57079999951 -0 0, axis 0 0 1, limit lower=-0.523595776 upper=0.523595776 effort=2.0 velocity=2.0
- added joint Head_J2_Joint: type revolute, parent Head_J1_Link, child Head_J2_Link, origin xyz=0 0 0 rpy=-1.57079999951 0 0, axis 0 0 1, limit lower=-1.57079633 upper=1.57079633 effort=2.0 velocity=2.0
- added joint world_to_base: type fixed, parent world, child base_link, origin xyz=0 0 0.0610021333 rpy=0 -0 0
- joint mount_L: parent base_link -> Gento_Luna_Leg_J6_Link
- joint mount_R: parent base_link -> Gento_Luna_Leg_J6_Link

Commit message: 更换手臂sdk ,优化逆解

File: ros2_ws/src/marvin_mesh_sim/urdf/marvin_mesh_hands.urdf (robot description, URDF)
Before this commit: robot marvin_whole_robot, 52 links, 51 joints
Links:
- removed link L_little_link1
- removed link L_little_link2
- removed link L_little_link3
- removed link R_little_link1
- removed link R_little_link2
- removed link R_little_link3
- added link L_ring_link1, mass 0.025089; collision box size=0.0304897754 0.0455897636 0.0380782186; visual mesh filename=package://marvin_mesh_sim/meshes/hands/left_hand/L_little_l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
- added link L_ring_link2, mass 0.11925; collision box size=0.0259896312 0.0699995552 0.0289999992; visual mesh filename=package://marvin_mesh_sim/meshes/hands/left_hand/L_little_l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
- added link L_ring_link3, mass 0.032861; collision box size=0.0267166012 0.0664134016 0.0287530166; visual mesh filename=package://marvin_mesh_sim/meshes/hands/left_hand/L_little_l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
- added link R_ring_link1, mass 0.025089; collision box size=0.0304897754 0.0455897636 0.0380782186; visual mesh filename=package://marvin_mesh_sim/meshes/hands/right_hand/R_little_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
- added link R_ring_link2, mass 0.11925; collision box size=0.0259896312 0.0699995552 0.0289999992; visual mesh filename=package://marvin_mesh_sim/meshes/hands/right_hand/R_little_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
- added link R_ring_link3, mass 0.03286; collision box size=0.0267166012 0.0664134016 0.0287530158; visual mesh filename=package://marvin_mesh_sim/meshes/hands/right_hand/R_little_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
Joints:
- removed joint L_index_j1
- removed joint L_index_j2
- removed joint L_index_j3
- removed joint L_little_j1
- removed joint L_little_j2
- removed joint L_little_j3
- removed joint L_middle_j1
- removed joint L_middle_j2
- removed joint L_thumb_j1
- removed joint L_thumb_j2
- removed joint L_thumb_j3
- removed joint R_index_j1
- removed joint R_index_j2
- removed joint R_index_j3
- removed joint R_little_j1
- removed joint R_little_j2
- removed joint R_little_j3
- removed joint R_middle_j1
- removed joint R_middle_j2
- removed joint R_thumb_j1
- removed joint R_thumb_j2
- removed joint R_thumb_j3
- added joint L_Joint1: type revolute, parent L_hand_base, child L_thumb_link1, origin xyz=-0.031492 -0.031853 0.0384 rpy=0 -0 0, axis 0 0 1, limit lower=0.0 upper=2.181661564992912 effort=2.0 velocity=2.0
- added joint L_Joint10: type revolute, parent L_ring_link1, child L_ring_link2, origin xyz=0.0205 0.024 0.0281 rpy=3.14159265359 1.57079265408 3.14159265359, axis 0 0 1, limit lower=0.0 upper=2.18 effort=2.0 velocity=2.0
- added joint L_Joint11: type revolute, parent L_ring_link2, child L_ring_link3, origin xyz=0 0.05 -0.001 rpy=0 -0 0, axis 0 0 1, limit lower=-1.0471975511965976 upper=1.57 effort=2.0 velocity=2.0
- added joint L_Joint2: type revolute, parent L_thumb_link1, child L_thumb_link2, origin xyz=-0.024 0.0155 0.0176 rpy=1.57079999951 -0 0, axis 0 0 -1, limit lower=-2.6179938779914944 upper=0.0 effort=2.0 velocity=2.0
- added joint L_Joint3: type revolute, parent L_thumb_link2, child L_thumb_link3, origin xyz=-0.026496 0.042402 0.001 rpy=0 -0 0, axis 0 0 -1, limit lower=-1.0471975511965976 upper=1.57 effort=2.0 velocity=2.0
- added joint L_Joint4: type revolute, parent L_hand_base, child L_index_link1, origin xyz=-0.0315 -0.020758 0.086 rpy=1.57079999951 -0 0, axis 0 0 -1, limit lower=-1.57 upper=0.0 effort=2.0 velocity=2.0
- added joint L_Joint5: type revolute, parent L_index_link1, child L_index_link2, origin xyz=0.0155 0.024 0.0281 rpy=3.14159265359 1.57079265408 3.14159265359, axis 0 0 1, limit lower=0.0 upper=2.18 effort=2.0 velocity=2.0
- added joint L_Joint6: type revolute, parent L_index_link2, child L_index_link3, origin xyz=0 0.05 -0.001 rpy=0 -0 0, axis 0 0 1, limit lower=-1.0471975511965976 upper=1.57 effort=2.0 velocity=2.0
- added joint L_Joint7: type revolute, parent L_hand_base, child L_middle_link1, origin xyz=0.018 -0.048858 0.1135 rpy=1.57080000079 -6.749156789e-12 1.57080000079, axis 0 0 1, limit lower=0.0 upper=2.18 effort=2.0 velocity=2.0
- added joint L_Joint8: type revolute, parent L_middle_link1, child L_middle_link2, origin xyz=0 0.05 -0.001 rpy=0 -0 0, axis 0 0 1, limit lower=-1.0471975511965976 upper=1.57 effort=2.0 velocity=2.0
- added joint L_Joint9: type revolute, parent L_hand_base, child L_ring_link1, origin xyz=0.0315 -0.020758 0.08 rpy=1.57079999951 -0 0, axis 0 0 -1, limit lower=0.0 upper=3.14 effort=2.0 velocity=2.0
- added joint R_Joint1: type revolute, parent R_hand_base, child R_thumb_link1, origin xyz=0.0315 -0.031858 0.0384 rpy=0 -0 0, axis 0 0 -1, limit lower=0.0 upper=2.181661564992912 effort=2.0 velocity=2.0
- added joint R_Joint10: type revolute, parent R_ring_link1, child R_ring_link2, origin xyz=-0.0205 0.024 0.0281 rpy=3.14159265359 1.57079265408 3.14159265359, axis 0 0 1, limit lower=0.0 upper=2.18 effort=2.0 velocity=2.0
- added joint R_Joint11: type revolute, parent R_ring_link2, child R_ring_link3, origin xyz=0 0.05 0.001 rpy=0 -0 0, axis 0 0 1, limit lower=-1.0471975511965976 upper=1.57 effort=2.0 velocity=2.0
- added joint R_Joint2: type revolute, parent R_thumb_link1, child R_thumb_link2, origin xyz=0.024 0.0155 0.0176 rpy=1.57079999951 -0 0, axis 0 0 1, limit lower=-2.6179938779914944 upper=0.0 effort=2.0 velocity=2.0
- added joint R_Joint3: type revolute, parent R_thumb_link2, child R_thumb_link3, origin xyz=0.026496 0.042402 0.001 rpy=0 -0 0, axis 0 0 1, limit lower=-1.0471975511965976 upper=1.57 effort=2.0 velocity=2.0
- added joint R_Joint4: type revolute, parent R_hand_base, child R_index_link1, origin xyz=0.0315000341 -0.0207580842 0.086 rpy=1.57079632679 -0 0, axis 0 0 1, limit lower=-1.57 upper=0.0 effort=2.0 velocity=2.0
- added joint R_Joint5: type revolute, parent R_index_link1, child R_index_link2, origin xyz=-0.0155 0.024 0.0281 rpy=3.14159265359 1.57079265408 3.14159265359, axis 0 0 1, limit lower=0.0 upper=2.18 effort=2.0 velocity=2.0
- added joint R_Joint6: type revolute, parent R_index_link2, child R_index_link3, origin xyz=0 0.05 0.001 rpy=0 -0 0, axis 0 0 1, limit lower=-1.0471975511965976 upper=1.57 effort=2.0 velocity=2.0
- added joint R_Joint7: type revolute, parent R_hand_base, child R_middle_link1, origin xyz=-0.018 -0.048858 0.1135 rpy=1.57080000079 -6.749156789e-12 1.57080000079, axis 0 0 1, limit lower=0.0 upper=2.18 effort=2.0 velocity=2.0
- added joint R_Joint8: type revolute, parent R_middle_link1, child R_middle_link2, origin xyz=0 0.05 0.001 rpy=0 -0 0, axis 0 0 1, limit lower=-1.0471975511965976 upper=1.57 effort=2.0 velocity=2.0
- added joint R_Joint9: type revolute, parent R_hand_base, child R_ring_link1, origin xyz=-0.0315 -0.020758 0.08 rpy=1.57079999951 -0 0, axis 0 0 1, limit lower=0.0 upper=3.14 effort=2.0 velocity=2.0

Commit message: feat: use palm-center TCP for dual-arm FK and IK

File: ros2_ws/src/marvin_mesh_sim/urdf/marvin_mesh_hands.urdf (robot description, URDF)
Before this commit: robot marvin_whole_robot, 52 links, 51 joints
Links:
- added link palm_center_L
- added link palm_center_R
Joints:
- added joint L_hand_base_to_palm_center: type fixed, parent L_hand_base, child palm_center_L, origin xyz=-6.64759427309e-05 -0.0166790671647 0.0625857863691 rpy=0 0 0
- added joint R_hand_base_to_palm_center: type fixed, parent R_hand_base, child palm_center_R, origin xyz=6.66882842779e-05 -0.0166790671647 0.0625857863691 rpy=0 0 0
